Commit message: Running Gazebo sim

File: urdf/ur5e.urdf.xacro (robot description, xacro)
@@ -78,13 +78,13 @@
       <visual>
         <geometry>
-          <mesh filename="package://ur5_arm/urdf/meshes/ur5e/visual/base.dae" />
-        </geometry>
-        <material name="LightGrey">
-          <color rgba="0.7 0.7 0.7 1.0"/>
-        </material>
-      </visual>
-      <collision>
-        <geometry>
-          <mesh filename="package://ur5_arm/urdf/meshes/ur5e/collision/base.stl" />
+          <mesh filename="model://ur5_arm/urdf/meshes/ur5e/visual/base.dae" />
+        </geometry>
+        <material name="LightGrey">
+          <color rgba="0.7 0.7 0.7 1.0"/>
+        </material>
+      </visual>
+      <collision>
+        <geometry>
+          <mesh filename="model://ur5_arm/urdf/meshes/ur5e/collision/base.stl" />
         </geometry>
       </collision>
@@ -115,13 +115,13 @@
       <visual>
         <geometry>
-          <mesh filename="package://ur5_arm/urdf/meshes/ur5e/visual/shoulder.dae" />
-        </geometry>
-        <material name="LightGrey">
-          <color rgba="0.7 0.7 0.7 1.0"/>
-        </material>
-      </visual>
-      <collision>
-        <geometry>
-          <mesh filename="package://ur5_arm/urdf/meshes/ur5e/collision/shoulder.stl" />
+          <mesh filename="model://ur5_arm/urdf/meshes/ur5e/visual/shoulder.dae" />
+        </geometry>
+        <material name="LightGrey">
+          <color rgba="0.7 0.7 0.7 1.0"/>
+        </material>
+      </visual>
+      <collision>
+        <geometry>
+          <mesh filename="model://ur5_arm/urdf/meshes/ur5e/collision/shoulder.stl" />
         </geometry>
       </collision>
@@ -152,13 +152,13 @@
       <visual>
         <geometry>
-          <mesh filename="package://ur5_arm/urdf/meshes/ur5e/visual/upperarm.dae" />
-        </geometry>
-        <material name="LightGrey">
-          <color rgba="0.7 0.7 0.7 1.0"/>
-        </material>
-      </visual>
-      <collision>
-        <geometry>
-          <mesh filename="package://ur5_arm/urdf/meshes/ur5e/collision/upperarm.stl" />
+          <mesh filename="model://ur5_arm/urdf/meshes/ur5e/visual/upperarm.dae" />
+        </geometry>
+        <material name="LightGrey">
+          <color rgba="0.7 0.7 0.7 1.0"/>
+        </material>
+      </visual>
+      <collision>
+        <geometry>
+          <mesh filename="model://ur5_arm/urdf/meshes/ur5e/collision/upperarm.stl" />
         </geometry>
       </collision>
@@ -189,13 +189,13 @@
       <visual>
         <geometry>
-          <mesh filename="package://ur5_arm/urdf/meshes/ur5e/visual/forearm.dae" />
-        </geometry>
-        <material name="LightGrey">
-          <color rgba="0.7 0.7 0.7 1.0"/>
-        </material>
-      </visual>
-      <collision>
-        <geometry>
-          <mesh filename="package://ur5_arm/urdf/meshes/ur5e/collision/forearm.stl" />
+          <mesh filename="model://ur5_arm/urdf/meshes/ur5e/visual/forearm.dae" />
+        </geometry>
+        <material name="LightGrey">
+          <color rgba="0.7 0.7 0.7 1.0"/>
+        </material>
+      </visual>
+      <collision>
+        <geometry>
+          <mesh filename="model://ur5_arm/urdf/meshes/ur5e/collision/forearm.stl" />
         </geometry>
       </collision>
@@ -226,13 +226,13 @@
       <visual>
         <geometry>
-          <mesh filename="package://ur5_arm/urdf/meshes/ur5e/visual/wrist1.dae" />
-        </geometry>
-        <material name="LightGrey">
-          <color rgba="0.7 0.7 0.7 1.0"/>
-        </material>
-      </visual>
-      <collision>
-        <geometry>
-          <mesh filename="package://ur5_arm/urdf/meshes/ur5e/collision/wrist1.stl" />
+          <mesh filename="model://ur5_arm/urdf/meshes/ur5e/visual/wrist1.dae" />
+        </geometry>
+        <material name="LightGrey">
+          <color rgba="0.7 0.7 0.7 1.0"/>
+        </material>
+      </visual>
+      <collision>
+        <geometry>
+          <mesh filename="model://ur5_arm/urdf/meshes/ur5e/collision/wrist1.stl" />
         </geometry>
       </collision>
@@ -263,13 +263,13 @@
       <visual>
         <geometry>
-          <mesh filename="package://ur5_arm/urdf/meshes/ur5e/visual/wrist2.dae" />
-        </geometry>
-        <material name="LightGrey">
-          <color rgba="0.7 0.7 0.7 1.0"/>
-        </material>
-      </visual>
-      <collision>
-        <geometry>
-          <mesh filename="package://ur5_arm/urdf/meshes/ur5e/collision/wrist2.stl" />
+          <mesh filename="model://ur5_arm/urdf/meshes/ur5e/visual/wrist2.dae" />
+        </geometry>
+        <material name="LightGrey">
+          <color rgba="0.7 0.7 0.7 1.0"/>
+        </material>
+      </visual>
+      <collision>
+        <geometry>
+          <mesh filename="model://ur5_arm/urdf/meshes/ur5e/collision/wrist2.stl" />
         </geometry>
       </collision>
@@ -300,13 +300,13 @@
       <visual>
         <geometry>
-          <mesh filename="package://ur5_arm/urdf/meshes/ur5e/visual/wrist3.dae" />
-        </geometry>
-        <material name="LightGrey">
-          <color rgba="0.7 0.7 0.7 1.0"/>
-        </material>
-      </visual>
-      <collision>
-        <geometry>
-          <mesh filename="package://ur5_arm/urdf/meshes/ur5e/collision/wrist3.stl" />
+          <mesh filename="model://ur5_arm/urdf/meshes/ur5e/visual/wrist3.dae" />
+        </geometry>
+        <material name="LightGrey">
+          <color rgba="0.7 0.7 0.7 1.0"/>
+        </material>
+      </visual>
+      <collision>
+        <geometry>
+          <mesh filename="model://ur5_arm/urdf/meshes/ur5e/collision/wrist3.stl" />
         </geometry>
       </collision>
