Commit message: Camera bridge added. Still need to fix its orientation

File: urdf/cam_support.urdf.xacro (robot description, xacro)
@@ -1,25 +1,6 @@
 <?xml version="1.0"?>
-<robot xmlns:xacro="http://ros.org/wiki/xacro" name="ur5e" >
-  <xacro:arg name="use_nominal_extrinsics" default="false"/>
-  <xacro:arg name="add_plug" default="true" />
-  <xacro:arg name="use_mesh" default="true" />
-  <!-- ur5e -->
-  <xacro:include filename="$(find ur5_arm)/urdf/ur5e.urdf.xacro" />
-  <xacro:include filename="$(find ur5_arm)/urdf/_d435.urdf.xacro" />
-  <!-- arm -->
-  <xacro:ur5e_robot prefix="" joint_limited="true"
-    shoulder_pan_lower_limit="${-pi}" shoulder_pan_upper_limit="${pi}"
-    shoulder_lift_lower_limit="${-pi}" shoulder_lift_upper_limit="${pi}"
-    elbow_joint_lower_limit="${-pi}" elbow_joint_upper_limit="${pi}"
-    wrist_1_lower_limit="${-pi}" wrist_1_upper_limit="${pi}"
-    wrist_2_lower_limit="${-pi}" wrist_2_upper_limit="${pi}"
-    wrist_3_lower_limit="${-pi}" wrist_3_upper_limit="${pi}"
-  />
-  <link name="world" />
-  <joint name="world_joint" type="fixed">
-    <parent link="world" />
-    <child link = "base_link" />
-    <origin xyz="0.0 0.0 0.0" rpy="0.0 0.0 0.0" />
-  </joint>
+<robot xmlns:xacro="http://ros.org/wiki/xacro" name="cam_support" >
+  <!-- Realsense d435 -->
+  <xacro:include filename="$(find ur5_weaver)/urdf/_d435.urdf.xacro" />
   <!-- Frame coincident with all-zeros TCP on UR controller -->
   <xacro:property name="tool0_offset" value="0.15"/>
@@ -45,9 +26,9 @@
   # CAN Support code
   ######################################## -->
-  <link name="webots_tool_link" />
-  <joint name="webots_tool_joint" type="fixed">
+  <link name="gz_tool_link" />
+  <joint name="gz_tool_joint" type="fixed">
     <origin rpy="1.57 0 0" xyz="0 0 0"/>
     <parent link="tool0"/>
-    <child link="webots_tool_link"/>
+    <child link="gz_tool_link"/>
   </joint>
   <!-- o wrist 2 fica 0.09465 m abaixo de wrist 3 (-0.0445+0.09465)-->
@@ -59,5 +40,5 @@
       <origin rpy="0 0 0" xyz="0 0 0"/>
       <geometry>
-        <mesh filename="package://ur5_arm/urdf/meshes/protos/CAM_Support2.stl" scale="1 1 1"/>
+        <mesh filename="package://ur5_weaver/meshes/protos/CAM_support.STL" scale="0.001 0.001 0.001"/>
       </geometry>
       <material name="Cyan">
@@ -68,18 +49,37 @@
   <joint name="CAM_support_joint" type="fixed">
     <origin rpy="0 -1.5704511 1.5705682" xyz="0.0447 -0.126 -0.0035"/>
-    <parent link="webots_tool_link"/>
+    <parent link="gz_tool_link"/>
     <child link="CAM_support_link"/>
   </joint>
-  <link name="camera_webots_link" />
-  <joint name="camera_webots_joint" type="fixed">
+  <link name="camera_gz_link" />
+  <joint name="camera_gz_joint" type="fixed">
     <origin rpy="0 1.5707963 -1.3090063" xyz="0.112 -0.093 0"/>
-    <parent link="webots_tool_link"/>
-    <child link="camera_webots_link"/>
+    <parent link="gz_tool_link"/>
+    <child link="camera_gz_link"/>
   </joint>
   <link name="camera_ros_link" />
   <joint name="camera_ros_joint" type="fixed">
     <origin rpy="0 3.14 3.14" xyz="0 0 0"/>
-    <parent link="camera_webots_link"/>
+    <parent link="camera_gz_link"/>
     <child link="camera_ros_link"/>
   </joint>
+  <gazebo reference="camera_ros_link">
+    <sensor name="camera" type="camera">
+      <camera>
+        <horizontal_fov>1.047</horizontal_fov>
+        <image>
+        <width>640</width>
+        <height>480</height>
+        </image>
+        <clip>
+        <near>0.1</near>
+        <far>100</far>
+        </clip>
+      </camera>
+      <always_on>1</always_on>
+      <update_rate>30</update_rate>
+      <visualize>true</visualize>
+      <topic>camera</topic>
+    </sensor>
+  </gazebo>
 </robot>

File: urdf/ur.urdf.xacro (robot description, xacro)
@@ -5,4 +5,5 @@
    <!-- import main macro -->
    <xacro:include filename="$(find ur5_weaver)/urdf/ur_macro.urdf.xacro"/>
+   <xacro:include filename="$(find ur5_weaver)/urdf/cam_support.urdf.xacro" />
    <!-- possible 'ur_type' values: ur3, ur3e, ur5, ur5e, ur7e, ur10, ur10e, ur12e, ur16e, ur15, ur20, ur30 -->
    <!-- the default value should raise an error in case this was called without defining the type -->

Commit message: Camera orientation fixed

File: urdf/cam_support.urdf.xacro (robot description, xacro)
@@ -60,5 +60,5 @@
   <link name="camera_ros_link" />
   <joint name="camera_ros_joint" type="fixed">
-    <origin rpy="0 3.14 3.14" xyz="0 0 0"/>
+    <origin rpy="0 1.570796 3.14159" xyz="0 0 0"/>
     <parent link="camera_gz_link"/>
     <child link="camera_ros_link"/>
