Commit message: rename the bringup package

File: src/weaver_bringup/urdf/cam_support.urdf.xacro (robot description, xacro)
@@ -2,5 +2,5 @@
 <robot xmlns:xacro="http://ros.org/wiki/xacro" name="cam_support" >
   <!-- Realsense d435 -->
-  <xacro:include filename="$(find ur5_weaver)/urdf/_d435.urdf.xacro" />
+  <xacro:include filename="$(find weaver_bringup)/urdf/_d435.urdf.xacro" />
   <!-- Frame coincident with all-zeros TCP on UR controller -->
   <xacro:property name="tool0_offset" value="0.15"/>
@@ -40,5 +40,5 @@
       <origin rpy="0 0 0" xyz="0 0 0"/>
       <geometry>
-        <mesh filename="package://ur5_weaver/meshes/protos/CAM_support.STL" scale="0.001 0.001 0.001"/>
+        <mesh filename="package://weaver_bringup/meshes/protos/CAM_support.STL" scale="0.001 0.001 0.001"/>
       </geometry>
       <material name="Cyan">

File: src/weaver_bringup/urdf/ur.srdf.xacro (robot description, xacro)
@@ -5,5 +5,5 @@
   <!-- parameters -->
   <xacro:arg name="prefix" default="" />
-  <xacro:include filename="$(find ur5_weaver)/urdf/ur_macro.srdf.xacro"/>
+  <xacro:include filename="$(find weaver_bringup)/urdf/ur_macro.srdf.xacro"/>
   <xacro:ur_srdf name="$(arg name)" prefix="$(arg prefix)"/>
 </robot>

File: src/weaver_bringup/urdf/ur.urdf.xacro (robot description, xacro)
@@ -4,6 +4,6 @@
    <xacro:arg name="name" default="ur"/>
    <!-- import main macro -->
-   <xacro:include filename="$(find ur5_weaver)/urdf/ur_macro.urdf.xacro"/>
-   <xacro:include filename="$(find ur5_weaver)/urdf/cam_support.urdf.xacro" />
+   <xacro:include filename="$(find weaver_bringup)/urdf/ur_macro.urdf.xacro"/>
+   <xacro:include filename="$(find weaver_bringup)/urdf/cam_support.urdf.xacro" />
    <!-- possible 'ur_type' values: ur3, ur3e, ur5, ur5e, ur7e, ur10, ur10e, ur12e, ur16e, ur15, ur20, ur30 -->
    <!-- the default value should raise an error in case this was called without defining the type -->
@@ -124,5 +124,5 @@
     <gazebo>
       <plugin filename="gz_ros2_control-system" name="gz_ros2_control::GazeboSimROS2ControlPlugin">
-        <parameters>$(find ur5_weaver)/config/ur_controllers.yaml</parameters>
+        <parameters>$(find weaver_bringup)/config/ur_controllers.yaml</parameters>
       </plugin>
     </gazebo>

File: src/weaver_bringup/urdf/ur_macro.urdf.xacro (robot description, xacro)
@@ -94,5 +94,5 @@
     <xacro:if value="${generate_ros2_control_tag}">
       <!-- ros2 control include -->
-      <xacro:include filename="$(find ur5_weaver)/urdf/ur.ros2_control.xacro" />
+      <xacro:include filename="$(find weaver_bringup)/urdf/ur.ros2_control.xacro" />
       <!-- ros2 control instance -->
       <xacro:ur_ros2_control
